File: Folder_Structure/Resources/Templates/Kicad Templates/Example project.kicad_pcb (KiCad board)
At the start: 2 copper layers, 65 x 56 mm, 5 parts, among them J1 GPIO

Commit message: Templates
Parts:
- removed J1: GPIO, Connector_PinSocket_2.54mm:PinSocket_2x20_P2.54mm_Vertical
- removed MH1, MH2, MH3, MH4: MountingHole_2.7mm_M2.5, MountingHole:MountingHole_2.7mm_M2.5
Other:
- board outline removed
- board text added: "0.0000 mm / 0.0000 mm"
- board text added: "368.8786 mm x 184.3120 mm"
- board text removed: "0.2000 mm / 0.0000 mm"
- board text removed: "65.0000 mm x 56.0000 mm"
- board text removed: "CAMERA (OPTIONAL)"
- board text removed: "DISPLAY (OPTIONAL)"
- board text removed: "Extend PCB edge 0.5mm if using SMT header"
- board text removed: "Green"
- board text removed: "PoE"
- board text removed: "RJ45"
- board text removed: "USB"
